File: LanguageCard.kicad_pcb (KiCad board)
At the start: 2 copper layers, 100 x 77.5 mm, 42 parts, among them J1 Apple II Expansion Bus, SW1 ROM ENABLE, U1 74LS86, U10 74LS06, U2 74LS08, U3 74LS175, U4 74LS32, U5 74LS08, U6 74LS08, U7 ROM F8 (2716/32)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

Commit message: Mudança de Layout
Parts:
- removed C8, C9: 100n, Capacitor_THT:C_Axial_L3.8mm_D2.6mm_P7.50mm_Horizontal
- removed JP2: DUAL ROM, Jumper:SolderJumper-2_P1.3mm_Open_RoundedPad1.0x1.5mm
- removed JP3: SPST, Jumper:SolderJumper-2_P1.3mm_Open_RoundedPad1.0x1.5mm
- removed R7, R8: 10k, Resistor_THT:R_Axial_DIN0207_L6.3mm_D2.5mm_P10.16mm_Horizontal
- removed the REF** at (218.4, 95.2)
- removed the REF** at (231.1, 95.2)
- removed the REF** at (231.1, 82.5)
- removed the REF** at (218.4, 82.5)
- removed the REF** at (241.3, 95.2)
- removed SW1: ROM ENABLE, MySwitch:SW_Lever_2P2T_Alcoswitch_AE203SD1
- removed U7Alt1: '64-'512, Package_DIP:DIP-28_W15.24mm
- added REF**: ROM Disabled, MySymbol:Jumper_SilkScreen, F.Cu at (168.9, 89.5)
- added REF**: ROM Enabled, MySymbol:Jumper_SilkScreen, F.Cu at (168.9, 87.0)
- C1: footprint Capacitor_THT:CP_Radial_D5.0mm_P2.50mm -> Capacitor_THT:CP_Radial_D8.0mm_P5.00mm
- C2, C3, C4, C5, C6, C7: value 100n -> .1μF; footprint Capacitor_THT:C_Axial_L3.8mm_D2.6mm_P7.50mm_Horizontal -> Capacitor_THT:C_Rect_L7.0mm_W2.0mm_P5.00mm
- JP1: value ROM Enable -> ROM EN; footprint Connector_PinHeader_2.54mm:PinHeader_2x03_P2.54mm_Vertical -> Connector_PinHeader_2.54mm:PinHeader_1x03_P2.54mm_Vertical
- U7: value ROM F8 (2716/32) -> ROM F8 (2716)
- moved C4 62.3 mm to (156.8, 54.6)
- moved C3 61.4 mm to (83.9, 44.5), turned to 0 degrees
- moved C7 51.9 mm to (120.7, 47.0), turned to 90 degrees
- moved C5 46.7 mm to (97.8, 87.0), turned to 180 degrees
- moved JP1 31.0 mm to (155.0, 87.6), turned to 90 degrees
- moved R6 29.6 mm to (165.7, 71.1), turned to 0 degrees
- moved C6 26.6 mm to (154.3, 81.3), turned to 90 degrees
- moved R2 13.1 mm to (95.2, 44.5), turned to 0 degrees
- moved R1 7.73 mm to (95.9, 29.2)
- moved U5 7.63 mm to (157.5, 67.3)
- moved U4 7.62 mm to (135.9, 67.3)
- moved U6 5.09 mm to (135.9, 82.5)
- moved U10 5.09 mm to (157.5, 82.5)
- moved D1 3.18 mm to (102.2, 31.8)
- moved C2 3.16 mm to (118.7, 34.2)
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Connections:
- net /~{ROMCE} renamed Net-(U7-~{CE}/PGM)
- JP1 pad 1: /ROMEN -> /ROMCE
- JP1 pad 2: unconnected-(JP1-Pin_2-Pad2) -> /ROM
- JP1 pad 3: /F8SEL -> GND
- U10 pad 11: /ROMEN -> /ROM
- U10 pad 3: /ROMEN -> /ROM
- U2 pad 6: /F8SEL -> /ROMCE
- U7 pad 21: /ROMA11/VPP/~{WE} -> +5V
Routing:
- net GND: track 42.8 -> 2827.7 mm, vias 0 -> 3
- net +5V: track 29.1 -> 441.9 mm
- net /ROMCE: track 0.00 -> 69.2 mm, vias 0 -> 1
- net /ROMEN: track 60.9 -> 0.00 mm
- net /ROMA11/VPP/~{WE}: track 55.4 -> 0.00 mm
- net /F8SEL: track 36.0 -> 0.00 mm, vias 1 -> 0
- net /~{R}/W: track 72.5 -> 45.1 mm
- net /ROM: track 0.00 -> 25.3 mm, vias 0 -> 1
- net /~{RESET}: track 29.0 -> 44.3 mm
- net /A1: track 166.6 -> 151.9 mm
- net /~{DEV}: track 83.7 -> 97.1 mm
- net /WE: track 112.1 -> 98.7 mm, vias 0 -> 2
- net /PHI0: track 33.2 -> 45.2 mm, vias 1 -> 0
- net /ROMEN2: track 11.7 -> 0.00 mm
- net /BR/W: track 113.1 -> 102.3 mm
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- removed copper zone on F.Cu, net +5V
- removed copper zone on B.Cu, net GND
Other:
- board text removed: "JLCJLCJLCJLC"
- board text removed: "JP1: If not using switch. (front view) 2K ROM: (JP2 open) >2K ROM: (JP2 short)"
- board text removed: "JP2: Short, and install DPDT switch (or use pair of jumpers on JP1) for ability to select two different F8 ROM images on a single (larger than 2K) ROM."
- board text removed: "JP3: Short if using an SPST switch that only connects outer two pins"
- board text removed: "SW1: Toggle switch. Miniature, Sub-miniature, or Ultra- miniature, right angle, SPDT. (Sub, Ultra-mini use JP1 pads) For SPST, short JP3. To switch between two different F8 ROM images on a single 4K or greater chip, short JP2 and use DPDT - must have center OFF (ON-OFF-ON) in order to disable."
- board text removed: "U7: Optional. 2K or larger (E)EPROM for overriding the logic board's F8 ROM. Enable using SW1 or JP1."
- board text removed: "rev ${REVISION}"
